File: OSED_Badge.kicad_pcb (KiCad board)
At the start: 2 copper layers, 111.6 x 119.9 mm, 20 parts, among them U1 NT3H1101W0FHKH

Commit message: Badge Update
Parts:
- added REF**: PCB, Shawn_PCB_Business_card:PCB, B.Cu at (224.0, 35.5)
- REF**: moved to B.Cu
- moved C1 83.4 mm to (186.0, 94.0)
- moved TP2 78.9 mm to (188.5, 129.0)
- moved R1 77.6 mm to (178.5, 94.0), turned to -90 degrees
- moved TP1 77.3 mm to (185.5, 129.0)
- moved TP4 72.6 mm to (182.5, 129.0)
- moved TP5 71.5 mm to (177.0, 129.0)
- moved TP3 68.0 mm to (179.5, 129.0)
- moved REF** 62.9 mm to (146.4, 41.3), turned to -45 degrees
Routing:
- net Net-(D1-A): track 24.1 -> 49.9 mm, vias 2 -> 4
- net Net-(D1-K): track 0.00 -> 2.41 mm
- net Net-(D4-K): track 0.00 -> 2.01 mm
- net GND: track 3.62 -> 5.60 mm
- net (no net): track 658.5 -> 657.4 mm
